Commit message: Add CI configuration, improve command mode handling, and enhance protocol support
- Introduced a CI workflow for automated testing on push and pull requests.
- Added command mode management to ensure only one interface is active per joint.
- Enhanced protocol handling with new parameter read/write capabilities.
- Updated README with new parameters and usage examples.
- Added tests for command mode validation and protocol functionality.

File: description/robstride_example.urdf.xacro (robot description, xacro)
@@ -3,4 +3,5 @@
   <xacro:arg name="can_tx_topic" default="to_can_bus"/>
   <xacro:arg name="can_rx_topic" default="from_can_bus"/>
+  <xacro:include filename="$(find robstride_ros2)/description/robstride_motor_profiles.xacro"/>
   <link name="base_link"/>
   <link name="robstride_link"/>
@@ -24,31 +25,11 @@
       <param name="shutdown_stop_interval_ms">20</param>
       <param name="shutdown_confirmation_timeout_ms">300</param>
+      <param name="startup_connection_timeout_ms">3000</param>
+      <param name="startup_confirmation_timeout_ms">500</param>
+      <param name="startup_retries">3</param>
     </hardware>
     <joint name="robstride_joint">
-      <param name="can_id">1</param>
-      <!-- Nonzero motor-side CAN watchdog. 4000 ticks = 200 ms on EduLite05. -->
-      <param name="can_timeout_ticks">4000</param>
-      <!-- RS05 example. Confirm these values against the exact motor/firmware manual. -->
-      <param name="position_min">-12.566370614359172</param>
-      <param name="position_max">12.566370614359172</param>
-      <param name="velocity_min">-50.0</param>
-      <param name="velocity_max">50.0</param>
-      <param name="effort_min">-5.5</param>
-      <param name="effort_max">5.5</param>
-      <param name="kp_max">500.0</param>
-      <param name="kd_max">5.0</param>
-      <param name="kp">30.0</param>
-      <param name="kd">1.0</param>
-      <param name="direction">1</param>
-      <param name="gear_ratio">1.0</param>
-      <param name="position_offset">0.0</param>
-      <command_interface name="position"/>
-      <command_interface name="velocity"/>
-      <command_interface name="effort"/>
-      <state_interface name="position"/>
-      <state_interface name="velocity"/>
-      <state_interface name="effort"/>
-      <state_interface name="temperature"/>
-      <state_interface name="fault"/>
+      <xacro:robstride_edulite05_params can_id="1" direction="1" kp="30.0" kd="1.0"/>
+      <xacro:robstride_joint_interfaces/>
     </joint>
   </ros2_control>

File: description/robstride_motor_profiles.xacro (robot description, xacro)
@@ -54,6 +54,6 @@
     <param name="kp">${kp}</param><param name="kd">${kd}</param><param name="direction">${direction}</param><param name="gear_ratio">${gear_ratio}</param><param name="position_offset">${position_offset}</param>
   </xacro:macro>
-  <xacro:macro name="robstride_edulite05_params" params="can_id direction:=1 gear_ratio:=9.0 position_offset:=0.0 kp:=30.0 kd:=1.0 can_timeout_ticks:=4000">
-    <!-- Wire ranges are motor-axis values; gear_ratio converts position/velocity at the ROS interface. -->
+  <xacro:macro name="robstride_edulite05_params" params="can_id direction:=1 gear_ratio:=1.0 position_offset:=0.0 kp:=30.0 kd:=1.0 can_timeout_ticks:=4000">
+    <!-- EduLite05 firmware reports an output-axis value calculated from its motor encoder. -->
     <param name="can_id">${can_id}</param><param name="can_timeout_ticks">${can_timeout_ticks}</param><param name="position_min">-12.566370614</param><param name="position_max">12.566370614</param>
     <param name="velocity_min">-50.0</param><param name="velocity_max">50.0</param><param name="effort_min">-6.0</param><param name="effort_max">6.0</param>
