Commit message: added english README fix xacro value

File: description/robstride_motor_profiles.xacro (robot description, xacro)
@@ -2,8 +2,9 @@
 <robot xmlns:xacro="http://www.ros.org/wiki/xacro" name="robstride_motor_profiles">
   <!--
-    MIT/private-protocol measurement ranges collected from RobStride manuals and the
-    open-source robstride reference implementation. The position limits here are
-    protocol limits; apply tighter mechanical limits in the surrounding robot model.
-    EduLite05 has a separate physical effort limit and protocol wire range.
+    Private-protocol Type 1/2 normalization ranges verified against the English
+    manuals dated July 13, 2026 in RobStride/Product_Information. These are wire
+    ranges, not recommended mechanical limits. Apply tighter limits in the robot
+    model. gear_ratio represents an additional robot transmission and does not
+    describe the actuator's built-in reduction stage.
   -->
   <xacro:macro name="robstride_joint_interfaces">
@@ -23,4 +24,10 @@
     <param name="kp">${kp}</param><param name="kd">${kd}</param><param name="direction">${direction}</param><param name="gear_ratio">${gear_ratio}</param><param name="position_offset">${position_offset}</param>
   </xacro:macro>
+  <xacro:macro name="robstride_rs01_params" params="can_id direction:=1 gear_ratio:=1.0 position_offset:=0.0 kp:=30.0 kd:=1.0 can_timeout_ticks:=4000">
+    <param name="can_id">${can_id}</param><param name="can_timeout_ticks">${can_timeout_ticks}</param><param name="position_min">-12.566370614</param><param name="position_max">12.566370614</param>
+    <param name="velocity_min">-44.0</param><param name="velocity_max">44.0</param><param name="effort_min">-17.0</param><param name="effort_max">17.0</param>
+    <param name="effort_wire_min">-17.0</param><param name="effort_wire_max">17.0</param><param name="kp_max">500.0</param><param name="kd_max">5.0</param>
+    <param name="kp">${kp}</param><param name="kd">${kd}</param><param name="direction">${direction}</param><param name="gear_ratio">${gear_ratio}</param><param name="position_offset">${position_offset}</param>
+  </xacro:macro>
   <xacro:macro name="robstride_rs02_params" params="can_id direction:=1 gear_ratio:=1.0 position_offset:=0.0 kp:=30.0 kd:=1.0 can_timeout_ticks:=4000">
     <param name="can_id">${can_id}</param><param name="can_timeout_ticks">${can_timeout_ticks}</param><param name="position_min">-12.566370614</param><param name="position_max">12.566370614</param>
@@ -29,5 +36,5 @@
     <param name="kp">${kp}</param><param name="kd">${kd}</param><param name="direction">${direction}</param><param name="gear_ratio">${gear_ratio}</param><param name="position_offset">${position_offset}</param>
   </xacro:macro>
-  <xacro:macro name="robstride_rs03_params" params="can_id direction:=1 gear_ratio:=1.0 position_offset:=0.0 kp:=100.0 kd:=5.0 can_timeout_ticks:=1200">
+  <xacro:macro name="robstride_rs03_params" params="can_id direction:=1 gear_ratio:=1.0 position_offset:=0.0 kp:=100.0 kd:=5.0 can_timeout_ticks:=4000">
     <param name="can_id">${can_id}</param><param name="can_timeout_ticks">${can_timeout_ticks}</param><param name="position_min">-12.566370614</param><param name="position_max">12.566370614</param>
     <param name="velocity_min">-20.0</param><param name="velocity_max">20.0</param><param name="effort_min">-60.0</param><param name="effort_max">60.0</param>
@@ -35,8 +42,7 @@
     <param name="kp">${kp}</param><param name="kd">${kd}</param><param name="direction">${direction}</param><param name="gear_ratio">${gear_ratio}</param><param name="position_offset">${position_offset}</param>
   </xacro:macro>
-  <xacro:macro name="robstride_rs04_params" params="can_id direction:=1 gear_ratio:=1.0 position_offset:=0.0 kp:=100.0 kd:=5.0 can_timeout_ticks:=2400">
-    <!-- RS04 values must be checked against the installed firmware manual. -->
+  <xacro:macro name="robstride_rs04_params" params="can_id direction:=1 gear_ratio:=1.0 position_offset:=0.0 kp:=100.0 kd:=5.0 can_timeout_ticks:=4000">
     <param name="can_id">${can_id}</param><param name="can_timeout_ticks">${can_timeout_ticks}</param><param name="position_min">-12.566370614</param><param name="position_max">12.566370614</param>
-    <param name="velocity_min">-20.0</param><param name="velocity_max">20.0</param><param name="effort_min">-120.0</param><param name="effort_max">120.0</param>
+    <param name="velocity_min">-15.0</param><param name="velocity_max">15.0</param><param name="effort_min">-120.0</param><param name="effort_max">120.0</param>
     <param name="effort_wire_min">-120.0</param><param name="effort_wire_max">120.0</param><param name="kp_max">5000.0</param><param name="kd_max">100.0</param>
     <param name="kp">${kp}</param><param name="kd">${kd}</param><param name="direction">${direction}</param><param name="gear_ratio">${gear_ratio}</param><param name="position_offset">${position_offset}</param>
@@ -51,9 +57,8 @@
     <param name="can_id">${can_id}</param><param name="can_timeout_ticks">${can_timeout_ticks}</param><param name="position_min">-12.566370614</param><param name="position_max">12.566370614</param>
     <param name="velocity_min">-50.0</param><param name="velocity_max">50.0</param><param name="effort_min">-36.0</param><param name="effort_max">36.0</param>
-    <param name="effort_wire_min">-36.0</param><param name="effort_wire_max">36.0</param><param name="kp_max">500.0</param><param name="kd_max">5.0</param>
+    <param name="effort_wire_min">-36.0</param><param name="effort_wire_max">36.0</param><param name="kp_max">5000.0</param><param name="kd_max">100.0</param>
     <param name="kp">${kp}</param><param name="kd">${kd}</param><param name="direction">${direction}</param><param name="gear_ratio">${gear_ratio}</param><param name="position_offset">${position_offset}</param>
   </xacro:macro>
   <xacro:macro name="robstride_edulite05_params" params="can_id direction:=1 gear_ratio:=1.0 position_offset:=0.0 kp:=30.0 kd:=1.0 can_timeout_ticks:=4000">
-    <!-- EduLite05 firmware reports an output-axis value calculated from its motor encoder. -->
     <param name="can_id">${can_id}</param><param name="can_timeout_ticks">${can_timeout_ticks}</param><param name="position_min">-12.566370614</param><param name="position_max">12.566370614</param>
     <param name="velocity_min">-50.0</param><param name="velocity_max">50.0</param><param name="effort_min">-6.0</param><param name="effort_max">6.0</param>

File: test/test_motor_profiles.urdf.xacro (robot description, xacro)
@@ -7,10 +7,11 @@
     </hardware>
     <joint name="rs00"><xacro:robstride_rs00_params can_id="1"/><xacro:robstride_joint_interfaces/></joint>
-    <joint name="rs02"><xacro:robstride_rs02_params can_id="2"/><xacro:robstride_joint_interfaces/></joint>
-    <joint name="rs03"><xacro:robstride_rs03_params can_id="3"/><xacro:robstride_joint_interfaces/></joint>
-    <joint name="rs04"><xacro:robstride_rs04_params can_id="4"/><xacro:robstride_joint_interfaces/></joint>
-    <joint name="rs05"><xacro:robstride_rs05_params can_id="5"/><xacro:robstride_joint_interfaces/></joint>
-    <joint name="rs06"><xacro:robstride_rs06_params can_id="6"/><xacro:robstride_joint_interfaces/></joint>
-    <joint name="edulite05"><xacro:robstride_edulite05_params can_id="7"/><xacro:robstride_joint_interfaces/></joint>
+    <joint name="rs01"><xacro:robstride_rs01_params can_id="2"/><xacro:robstride_joint_interfaces/></joint>
+    <joint name="rs02"><xacro:robstride_rs02_params can_id="3"/><xacro:robstride_joint_interfaces/></joint>
+    <joint name="rs03"><xacro:robstride_rs03_params can_id="4"/><xacro:robstride_joint_interfaces/></joint>
+    <joint name="rs04"><xacro:robstride_rs04_params can_id="5"/><xacro:robstride_joint_interfaces/></joint>
+    <joint name="rs05"><xacro:robstride_rs05_params can_id="6"/><xacro:robstride_joint_interfaces/></joint>
+    <joint name="rs06"><xacro:robstride_rs06_params can_id="7"/><xacro:robstride_joint_interfaces/></joint>
+    <joint name="edulite05"><xacro:robstride_edulite05_params can_id="8"/><xacro:robstride_joint_interfaces/></joint>
   </ros2_control>
 </robot>
