Commit message: Require explicit motor gains

File: robstride_examples/description/robstride_motor_profiles.xacro (robot description, xacro)
@@ -18,5 +18,5 @@
     <state_interface name="fault"/>
   </xacro:macro>
-  <xacro:macro name="robstride_rs00_params" params="can_id direction:=1 gear_ratio:=1.0 position_offset:=0.0 kp:=30.0 kd:=1.0 can_timeout_ticks:=4000">
+  <xacro:macro name="robstride_rs00_params" params="can_id kp kd direction:=1 gear_ratio:=1.0 position_offset:=0.0 can_timeout_ticks:=4000">
     <param name="can_id">${can_id}</param><param name="can_timeout_ticks">${can_timeout_ticks}</param><param name="position_min">-12.566370614</param><param name="position_max">12.566370614</param>
     <param name="velocity_min">-33.0</param><param name="velocity_max">33.0</param><param name="effort_min">-14.0</param><param name="effort_max">14.0</param>
@@ -24,5 +24,5 @@
     <param name="kp">${kp}</param><param name="kd">${kd}</param><param name="direction">${direction}</param><param name="gear_ratio">${gear_ratio}</param><param name="position_offset">${position_offset}</param>
   </xacro:macro>
-  <xacro:macro name="robstride_rs01_params" params="can_id direction:=1 gear_ratio:=1.0 position_offset:=0.0 kp:=30.0 kd:=1.0 can_timeout_ticks:=4000">
+  <xacro:macro name="robstride_rs01_params" params="can_id kp kd direction:=1 gear_ratio:=1.0 position_offset:=0.0 can_timeout_ticks:=4000">
     <param name="can_id">${can_id}</param><param name="can_timeout_ticks">${can_timeout_ticks}</param><param name="position_min">-12.566370614</param><param name="position_max">12.566370614</param>
     <param name="velocity_min">-44.0</param><param name="velocity_max">44.0</param><param name="effort_min">-17.0</param><param name="effort_max">17.0</param>
@@ -30,5 +30,5 @@
     <param name="kp">${kp}</param><param name="kd">${kd}</param><param name="direction">${direction}</param><param name="gear_ratio">${gear_ratio}</param><param name="position_offset">${position_offset}</param>
   </xacro:macro>
-  <xacro:macro name="robstride_rs02_params" params="can_id direction:=1 gear_ratio:=1.0 position_offset:=0.0 kp:=30.0 kd:=1.0 can_timeout_ticks:=4000">
+  <xacro:macro name="robstride_rs02_params" params="can_id kp kd direction:=1 gear_ratio:=1.0 position_offset:=0.0 can_timeout_ticks:=4000">
     <param name="can_id">${can_id}</param><param name="can_timeout_ticks">${can_timeout_ticks}</param><param name="position_min">-12.566370614</param><param name="position_max">12.566370614</param>
     <param name="velocity_min">-44.0</param><param name="velocity_max">44.0</param><param name="effort_min">-17.0</param><param name="effort_max">17.0</param>
@@ -36,5 +36,5 @@
     <param name="kp">${kp}</param><param name="kd">${kd}</param><param name="direction">${direction}</param><param name="gear_ratio">${gear_ratio}</param><param name="position_offset">${position_offset}</param>
   </xacro:macro>
-  <xacro:macro name="robstride_rs03_params" params="can_id direction:=1 gear_ratio:=1.0 position_offset:=0.0 kp:=100.0 kd:=5.0 can_timeout_ticks:=4000">
+  <xacro:macro name="robstride_rs03_params" params="can_id kp kd direction:=1 gear_ratio:=1.0 position_offset:=0.0 can_timeout_ticks:=4000">
     <param name="can_id">${can_id}</param><param name="can_timeout_ticks">${can_timeout_ticks}</param><param name="position_min">-12.566370614</param><param name="position_max">12.566370614</param>
     <param name="velocity_min">-20.0</param><param name="velocity_max">20.0</param><param name="effort_min">-60.0</param><param name="effort_max">60.0</param>
@@ -42,5 +42,5 @@
     <param name="kp">${kp}</param><param name="kd">${kd}</param><param name="direction">${direction}</param><param name="gear_ratio">${gear_ratio}</param><param name="position_offset">${position_offset}</param>
   </xacro:macro>
-  <xacro:macro name="robstride_rs04_params" params="can_id direction:=1 gear_ratio:=1.0 position_offset:=0.0 kp:=100.0 kd:=5.0 can_timeout_ticks:=4000">
+  <xacro:macro name="robstride_rs04_params" params="can_id kp kd direction:=1 gear_ratio:=1.0 position_offset:=0.0 can_timeout_ticks:=4000">
     <param name="can_id">${can_id}</param><param name="can_timeout_ticks">${can_timeout_ticks}</param><param name="position_min">-12.566370614</param><param name="position_max">12.566370614</param>
     <param name="velocity_min">-15.0</param><param name="velocity_max">15.0</param><param name="effort_min">-120.0</param><param name="effort_max">120.0</param>
@@ -48,5 +48,5 @@
     <param name="kp">${kp}</param><param name="kd">${kd}</param><param name="direction">${direction}</param><param name="gear_ratio">${gear_ratio}</param><param name="position_offset">${position_offset}</param>
   </xacro:macro>
-  <xacro:macro name="robstride_rs05_params" params="can_id direction:=1 gear_ratio:=1.0 position_offset:=0.0 kp:=30.0 kd:=1.0 can_timeout_ticks:=4000">
+  <xacro:macro name="robstride_rs05_params" params="can_id kp kd direction:=1 gear_ratio:=1.0 position_offset:=0.0 can_timeout_ticks:=4000">
     <param name="can_id">${can_id}</param><param name="can_timeout_ticks">${can_timeout_ticks}</param><param name="position_min">-12.566370614</param><param name="position_max">12.566370614</param>
     <param name="velocity_min">-50.0</param><param name="velocity_max">50.0</param><param name="effort_min">-5.5</param><param name="effort_max">5.5</param>
@@ -54,5 +54,5 @@
     <param name="kp">${kp}</param><param name="kd">${kd}</param><param name="direction">${direction}</param><param name="gear_ratio">${gear_ratio}</param><param name="position_offset">${position_offset}</param>
   </xacro:macro>
-  <xacro:macro name="robstride_rs06_params" params="can_id direction:=1 gear_ratio:=1.0 position_offset:=0.0 kp:=30.0 kd:=1.0 can_timeout_ticks:=4000">
+  <xacro:macro name="robstride_rs06_params" params="can_id kp kd direction:=1 gear_ratio:=1.0 position_offset:=0.0 can_timeout_ticks:=4000">
     <param name="can_id">${can_id}</param><param name="can_timeout_ticks">${can_timeout_ticks}</param><param name="position_min">-12.566370614</param><param name="position_max">12.566370614</param>
     <param name="velocity_min">-50.0</param><param name="velocity_max">50.0</param><param name="effort_min">-36.0</param><param name="effort_max">36.0</param>
@@ -60,5 +60,5 @@
     <param name="kp">${kp}</param><param name="kd">${kd}</param><param name="direction">${direction}</param><param name="gear_ratio">${gear_ratio}</param><param name="position_offset">${position_offset}</param>
   </xacro:macro>
-  <xacro:macro name="robstride_edulite05_params" params="can_id direction:=1 gear_ratio:=1.0 position_offset:=0.0 kp:=30.0 kd:=1.0 can_timeout_ticks:=4000">
+  <xacro:macro name="robstride_edulite05_params" params="can_id kp kd direction:=1 gear_ratio:=1.0 position_offset:=0.0 can_timeout_ticks:=4000">
     <param name="can_id">${can_id}</param><param name="can_timeout_ticks">${can_timeout_ticks}</param><param name="position_min">-12.566370614</param><param name="position_max">12.566370614</param>
     <param name="velocity_min">-50.0</param><param name="velocity_max">50.0</param><param name="effort_min">-6.0</param><param name="effort_max">6.0</param>

File: robstride_examples/test/test_motor_profiles.urdf.xacro (robot description, xacro)
@@ -6,12 +6,12 @@
       <plugin>robstride_ros2/RobStrideSystem</plugin>
     </hardware>
-    <joint name="rs00"><xacro:robstride_rs00_params can_id="1"/><xacro:robstride_joint_interfaces/></joint>
-    <joint name="rs01"><xacro:robstride_rs01_params can_id="2"/><xacro:robstride_joint_interfaces/></joint>
-    <joint name="rs02"><xacro:robstride_rs02_params can_id="3"/><xacro:robstride_joint_interfaces/></joint>
-    <joint name="rs03"><xacro:robstride_rs03_params can_id="4"/><xacro:robstride_joint_interfaces/></joint>
-    <joint name="rs04"><xacro:robstride_rs04_params can_id="5"/><xacro:robstride_joint_interfaces/></joint>
-    <joint name="rs05"><xacro:robstride_rs05_params can_id="6"/><xacro:robstride_joint_interfaces/></joint>
-    <joint name="rs06"><xacro:robstride_rs06_params can_id="7"/><xacro:robstride_joint_interfaces/></joint>
-    <joint name="edulite05"><xacro:robstride_edulite05_params can_id="8"/><xacro:robstride_joint_interfaces/></joint>
+    <joint name="rs00"><xacro:robstride_rs00_params can_id="1" kp="30.0" kd="1.0"/><xacro:robstride_joint_interfaces/></joint>
+    <joint name="rs01"><xacro:robstride_rs01_params can_id="2" kp="30.0" kd="1.0"/><xacro:robstride_joint_interfaces/></joint>
+    <joint name="rs02"><xacro:robstride_rs02_params can_id="3" kp="30.0" kd="1.0"/><xacro:robstride_joint_interfaces/></joint>
+    <joint name="rs03"><xacro:robstride_rs03_params can_id="4" kp="100.0" kd="5.0"/><xacro:robstride_joint_interfaces/></joint>
+    <joint name="rs04"><xacro:robstride_rs04_params can_id="5" kp="100.0" kd="5.0"/><xacro:robstride_joint_interfaces/></joint>
+    <joint name="rs05"><xacro:robstride_rs05_params can_id="6" kp="30.0" kd="1.0"/><xacro:robstride_joint_interfaces/></joint>
+    <joint name="rs06"><xacro:robstride_rs06_params can_id="7" kp="30.0" kd="1.0"/><xacro:robstride_joint_interfaces/></joint>
+    <joint name="edulite05"><xacro:robstride_edulite05_params can_id="8" kp="30.0" kd="1.0"/><xacro:robstride_joint_interfaces/></joint>
   </ros2_control>
 </robot>

Commit message: Add operational command limits

File: robstride_examples/description/robstride_motor_profiles.xacro (robot description, xacro)
@@ -18,51 +18,67 @@
     <state_interface name="fault"/>
   </xacro:macro>
-  <xacro:macro name="robstride_rs00_params" params="can_id direction:=1 gear_ratio:=1.0 position_offset:=0.0 kp:=30.0 kd:=1.0 can_timeout_ticks:=4000">
+  <xacro:macro name="robstride_command_limits" params="position_min position_max velocity_min velocity_max effort_min effort_max">
+    <xacro:if value="${position_min != ''}"><param name="command_position_min">${position_min}</param></xacro:if>
+    <xacro:if value="${position_max != ''}"><param name="command_position_max">${position_max}</param></xacro:if>
+    <xacro:if value="${velocity_min != ''}"><param name="command_velocity_min">${velocity_min}</param></xacro:if>
+    <xacro:if value="${velocity_max != ''}"><param name="command_velocity_max">${velocity_max}</param></xacro:if>
+    <xacro:if value="${effort_min != ''}"><param name="command_effort_min">${effort_min}</param></xacro:if>
+    <xacro:if value="${effort_max != ''}"><param name="command_effort_max">${effort_max}</param></xacro:if>
+  </xacro:macro>
+  <xacro:macro name="robstride_rs00_params" params="can_id direction:=1 gear_ratio:=1.0 position_offset:=0.0 kp:=30.0 kd:=1.0 can_timeout_ticks:=4000 command_position_min:='' command_position_max:='' command_velocity_min:='' command_velocity_max:='' command_effort_min:='' command_effort_max:=''">
     <param name="can_id">${can_id}</param><param name="can_timeout_ticks">${can_timeout_ticks}</param><param name="position_min">-12.566370614</param><param name="position_max">12.566370614</param>
     <param name="velocity_min">-33.0</param><param name="velocity_max">33.0</param><param name="effort_min">-14.0</param><param name="effort_max">14.0</param>
     <param name="effort_wire_min">-14.0</param><param name="effort_wire_max">14.0</param><param name="kp_max">500.0</param><param name="kd_max">5.0</param>
     <param name="kp">${kp}</param><param name="kd">${kd}</param><param name="direction">${direction}</param><param name="gear_ratio">${gear_ratio}</param><param name="position_offset">${position_offset}</param>
+    <xacro:robstride_command_limits position_min="${command_position_min}" position_max="${command_position_max}" velocity_min="${command_velocity_min}" velocity_max="${command_velocity_max}" effort_min="${command_effort_min}" effort_max="${command_effort_max}"/>
   </xacro:macro>
-  <xacro:macro name="robstride_rs01_params" params="can_id direction:=1 gear_ratio:=1.0 position_offset:=0.0 kp:=30.0 kd:=1.0 can_timeout_ticks:=4000">
+  <xacro:macro name="robstride_rs01_params" params="can_id direction:=1 gear_ratio:=1.0 position_offset:=0.0 kp:=30.0 kd:=1.0 can_timeout_ticks:=4000 command_position_min:='' command_position_max:='' command_velocity_min:='' command_velocity_max:='' command_effort_min:='' command_effort_max:=''">
     <param name="can_id">${can_id}</param><param name="can_timeout_ticks">${can_timeout_ticks}</param><param name="position_min">-12.566370614</param><param name="position_max">12.566370614</param>
     <param name="velocity_min">-44.0</param><param name="velocity_max">44.0</param><param name="effort_min">-17.0</param><param name="effort_max">17.0</param>
     <param name="effort_wire_min">-17.0</param><param name="effort_wire_max">17.0</param><param name="kp_max">500.0</param><param name="kd_max">5.0</param>
     <param name="kp">${kp}</param><param name="kd">${kd}</param><param name="direction">${direction}</param><param name="gear_ratio">${gear_ratio}</param><param name="position_offset">${position_offset}</param>
+    <xacro:robstride_command_limits position_min="${command_position_min}" position_max="${command_position_max}" velocity_min="${command_velocity_min}" velocity_max="${command_velocity_max}" effort_min="${command_effort_min}" effort_max="${command_effort_max}"/>
   </xacro:macro>
-  <xacro:macro name="robstride_rs02_params" params="can_id direction:=1 gear_ratio:=1.0 position_offset:=0.0 kp:=30.0 kd:=1.0 can_timeout_ticks:=4000">
+  <xacro:macro name="robstride_rs02_params" params="can_id direction:=1 gear_ratio:=1.0 position_offset:=0.0 kp:=30.0 kd:=1.0 can_timeout_ticks:=4000 command_position_min:='' command_position_max:='' command_velocity_min:='' command_velocity_max:='' command_effort_min:='' command_effort_max:=''">
     <param name="can_id">${can_id}</param><param name="can_timeout_ticks">${can_timeout_ticks}</param><param name="position_min">-12.566370614</param><param name="position_max">12.566370614</param>
     <param name="velocity_min">-44.0</param><param name="velocity_max">44.0</param><param name="effort_min">-17.0</param><param name="effort_max">17.0</param>
     <param name="effort_wire_min">-17.0</param><param name="effort_wire_max">17.0</param><param name="kp_max">500.0</param><param name="kd_max">5.0</param>
     <param name="kp">${kp}</param><param name="kd">${kd}</param><param name="direction">${direction}</param><param name="gear_ratio">${gear_ratio}</param><param name="position_offset">${position_offset}</param>
+    <xacro:robstride_command_limits position_min="${command_position_min}" position_max="${command_position_max}" velocity_min="${command_velocity_min}" velocity_max="${command_velocity_max}" effort_min="${command_effort_min}" effort_max="${command_effort_max}"/>
   </xacro:macro>
-  <xacro:macro name="robstride_rs03_params" params="can_id direction:=1 gear_ratio:=1.0 position_offset:=0.0 kp:=100.0 kd:=5.0 can_timeout_ticks:=4000">
+  <xacro:macro name="robstride_rs03_params" params="can_id direction:=1 gear_ratio:=1.0 position_offset:=0.0 kp:=100.0 kd:=5.0 can_timeout_ticks:=4000 command_position_min:='' command_position_max:='' command_velocity_min:='' command_velocity_max:='' command_effort_min:='' command_effort_max:=''">
     <param name="can_id">${can_id}</param><param name="can_timeout_ticks">${can_timeout_ticks}</param><param name="position_min">-12.566370614</param><param name="position_max">12.566370614</param>
     <param name="velocity_min">-20.0</param><param name="velocity_max">20.0</param><param name="effort_min">-60.0</param><param name="effort_max">60.0</param>
     <param name="effort_wire_min">-60.0</param><param name="effort_wire_max">60.0</param><param name="kp_max">5000.0</param><param name="kd_max">100.0</param>
     <param name="kp">${kp}</param><param name="kd">${kd}</param><param name="direction">${direction}</param><param name="gear_ratio">${gear_ratio}</param><param name="position_offset">${position_offset}</param>
+    <xacro:robstride_command_limits position_min="${command_position_min}" position_max="${command_position_max}" velocity_min="${command_velocity_min}" velocity_max="${command_velocity_max}" effort_min="${command_effort_min}" effort_max="${command_effort_max}"/>
   </xacro:macro>
-  <xacro:macro name="robstride_rs04_params" params="can_id direction:=1 gear_ratio:=1.0 position_offset:=0.0 kp:=100.0 kd:=5.0 can_timeout_ticks:=4000">
+  <xacro:macro name="robstride_rs04_params" params="can_id direction:=1 gear_ratio:=1.0 position_offset:=0.0 kp:=100.0 kd:=5.0 can_timeout_ticks:=4000 command_position_min:='' command_position_max:='' command_velocity_min:='' command_velocity_max:='' command_effort_min:='' command_effort_max:=''">
     <param name="can_id">${can_id}</param><param name="can_timeout_ticks">${can_timeout_ticks}</param><param name="position_min">-12.566370614</param><param name="position_max">12.566370614</param>
     <param name="velocity_min">-15.0</param><param name="velocity_max">15.0</param><param name="effort_min">-120.0</param><param name="effort_max">120.0</param>
     <param name="effort_wire_min">-120.0</param><param name="effort_wire_max">120.0</param><param name="kp_max">5000.0</param><param name="kd_max">100.0</param>
     <param name="kp">${kp}</param><param name="kd">${kd}</param><param name="direction">${direction}</param><param name="gear_ratio">${gear_ratio}</param><param name="position_offset">${position_offset}</param>
+    <xacro:robstride_command_limits position_min="${command_position_min}" position_max="${command_position_max}" velocity_min="${command_velocity_min}" velocity_max="${command_velocity_max}" effort_min="${command_effort_min}" effort_max="${command_effort_max}"/>
   </xacro:macro>
-  <xacro:macro name="robstride_rs05_params" params="can_id direction:=1 gear_ratio:=1.0 position_offset:=0.0 kp:=30.0 kd:=1.0 can_timeout_ticks:=4000">
+  <xacro:macro name="robstride_rs05_params" params="can_id direction:=1 gear_ratio:=1.0 position_offset:=0.0 kp:=30.0 kd:=1.0 can_timeout_ticks:=4000 command_position_min:='' command_position_max:='' command_velocity_min:='' command_velocity_max:='' command_effort_min:='' command_effort_max:=''">
     <param name="can_id">${can_id}</param><param name="can_timeout_ticks">${can_timeout_ticks}</param><param name="position_min">-12.566370614</param><param name="position_max">12.566370614</param>
     <param name="velocity_min">-50.0</param><param name="velocity_max">50.0</param><param name="effort_min">-5.5</param><param name="effort_max">5.5</param>
     <param name="effort_wire_min">-5.5</param><param name="effort_wire_max">5.5</param><param name="kp_max">500.0</param><param name="kd_max">5.0</param>
     <param name="kp">${kp}</param><param name="kd">${kd}</param><param name="direction">${direction}</param><param name="gear_ratio">${gear_ratio}</param><param name="position_offset">${position_offset}</param>
+    <xacro:robstride_command_limits position_min="${command_position_min}" position_max="${command_position_max}" velocity_min="${command_velocity_min}" velocity_max="${command_velocity_max}" effort_min="${command_effort_min}" effort_max="${command_effort_max}"/>
   </xacro:macro>
-  <xacro:macro name="robstride_rs06_params" params="can_id direction:=1 gear_ratio:=1.0 position_offset:=0.0 kp:=30.0 kd:=1.0 can_timeout_ticks:=4000">
+  <xacro:macro name="robstride_rs06_params" params="can_id direction:=1 gear_ratio:=1.0 position_offset:=0.0 kp:=30.0 kd:=1.0 can_timeout_ticks:=4000 command_position_min:='' command_position_max:='' command_velocity_min:='' command_velocity_max:='' command_effort_min:='' command_effort_max:=''">
     <param name="can_id">${can_id}</param><param name="can_timeout_ticks">${can_timeout_ticks}</param><param name="position_min">-12.566370614</param><param name="position_max">12.566370614</param>
     <param name="velocity_min">-50.0</param><param name="velocity_max">50.0</param><param name="effort_min">-36.0</param><param name="effort_max">36.0</param>
     <param name="effort_wire_min">-36.0</param><param name="effort_wire_max">36.0</param><param name="kp_max">5000.0</param><param name="kd_max">100.0</param>
     <param name="kp">${kp}</param><param name="kd">${kd}</param><param name="direction">${direction}</param><param name="gear_ratio">${gear_ratio}</param><param name="position_offset">${position_offset}</param>
+    <xacro:robstride_command_limits position_min="${command_position_min}" position_max="${command_position_max}" velocity_min="${command_velocity_min}" velocity_max="${command_velocity_max}" effort_min="${command_effort_min}" effort_max="${command_effort_max}"/>
   </xacro:macro>
-  <xacro:macro name="robstride_edulite05_params" params="can_id direction:=1 gear_ratio:=1.0 position_offset:=0.0 kp:=30.0 kd:=1.0 can_timeout_ticks:=4000">
+  <xacro:macro name="robstride_edulite05_params" params="can_id direction:=1 gear_ratio:=1.0 position_offset:=0.0 kp:=30.0 kd:=1.0 can_timeout_ticks:=4000 command_position_min:='' command_position_max:='' command_velocity_min:='' command_velocity_max:='' command_effort_min:='' command_effort_max:=''">
     <param name="can_id">${can_id}</param><param name="can_timeout_ticks">${can_timeout_ticks}</param><param name="position_min">-12.566370614</param><param name="position_max">12.566370614</param>
     <param name="velocity_min">-50.0</param><param name="velocity_max">50.0</param><param name="effort_min">-6.0</param><param name="effort_max">6.0</param>
     <param name="effort_wire_min">-6.0</param><param name="effort_wire_max">6.0</param><param name="kp_max">500.0</param><param name="kd_max">5.0</param>
     <param name="kp">${kp}</param><param name="kd">${kd}</param><param name="direction">${direction}</param><param name="gear_ratio">${gear_ratio}</param><param name="position_offset">${position_offset}</param>
+    <xacro:robstride_command_limits position_min="${command_position_min}" position_max="${command_position_max}" velocity_min="${command_velocity_min}" velocity_max="${command_velocity_max}" effort_min="${command_effort_min}" effort_max="${command_effort_max}"/>
   </xacro:macro>
 </robot>
